File: controller/controller.sch (EAGLE design)
At the start: 8 parts, among them IC1 L297, IC2 L298, IC4 ATTINY24/44/84-PU

Commit message: Controllerschaltung weitergebaut
Parts:
- removed IC4: ATTINY24/44/84-PU, attiny24_44_84:ATTINY24/44/84-PU
- added SV1, SV2: (no value), con-lstb:MA06-1
- added X1: (no value), con-molex:22-23-2061
Connections:
- new net CLOCK: IC1.CLOCK, SV1.5
- new net CNTL: IC1.CNTL, SV2.4
- new net CW_CCW: IC1.CW/CCW, SV1.6
- new net DRV_RST: IC1.RESET, SV1.2
- new net ENABLE: IC1.ENABLE, SV2.5
- new net HOME: IC1.HOME, SV1.3
- new net H_F: IC1.H/F, SV1.4
- new net N$22: SV2.2
- new net VREF: IC1.VREF, SV2.3
- net +12V: now also IC3A.DC1+, IC3A.DC2+, IC3B.DC1+, IC3B.DC2+, SV1.1
- net GND: now also IC3A.DC1-, IC3A.DC2-, IC3B.DC1-, IC3B.DC2-, SV2.1; no longer IC4.GND
- net N$10: now also X1-2.S
- net N$11: now also X1-4.S
- net N$12: now also X1-3.S
- net N$9: now also X1-1.S
- net VCC: now also SV2.6; no longer IC1.ENABLE, IC4.VCC
